File: Hardware/Qwiic_ADS1219.kicad_pcb (KiCad board)
At the start: 2 copper layers, 25.4 x 25.4 mm, 30 parts, among them J1 Qwiic_RA, J2 Qwiic_RA, J3 Conn_01x06, J4 Conn_01x06, J5 Conn_01x02, J6 I2C_01x04, U1 ADS1219IPW

Commit message: Routed
Parts:
- added G***: LOGO, SparkFun-Aesthetic:qwiic_5.5mm, F.Cu at (130.3, 109.0)
- added R4: 10k, SparkFun-Resistor:R_0603_1608Metric, F.Cu at (144.8, 113.7)
- added R5: 10k, SparkFun-Resistor:R_0603_1608Metric, F.Cu at (134.6, 113.7)
- added Ref**: Val**, SparkFun-Aesthetic:OSHW-LOGO-MINI, F.Cu at (150.0, 108.8)
- added kibuzzard-64C36D1A: G***, kibuzzard-64C36D1A, F.Cu at (134.6, 108.6)
- added kibuzzard-64C36D2D: G***, kibuzzard-64C36D2D, F.Cu at (137.2, 108.6)
- added kibuzzard-64C36D47: G***, kibuzzard-64C36D47, F.Cu at (139.7, 108.7)
- added kibuzzard-64C36D5B: G***, kibuzzard-64C36D5B, F.Cu at (142.2, 108.7)
- added kibuzzard-64C36D6C: G***, kibuzzard-64C36D6C, F.Cu at (144.8, 108.5)
- added kibuzzard-64C36D91: G***, kibuzzard-64C36D91, F.Cu at (147.3, 108.6)
- added kibuzzard-64C36E7A: G***, kibuzzard-64C36E7A, F.Cu at (133.3, 122.8)
- added kibuzzard-64C36E7A: G***, kibuzzard-64C36E7A, B.Cu at (138.4, 108.3)
- added kibuzzard-64C36E7A: G***, kibuzzard-64C36E7A, B.Cu at (133.3, 108.3)
- added kibuzzard-64C36E7A: G***, kibuzzard-64C36E7A, B.Cu at (146.1, 108.3)
- added kibuzzard-64C36E7A: G***, kibuzzard-64C36E7A, B.Cu at (135.9, 108.3)
- added kibuzzard-64C36E7A: G***, kibuzzard-64C36E7A, B.Cu at (133.3, 122.8)
- added kibuzzard-64C36E7A: G***, kibuzzard-64C36E7A, B.Cu at (143.5, 108.3)
- added kibuzzard-64C36EF5: G***, kibuzzard-64C36EF5, B.Cu at (141.0, 108.9)
- added kibuzzard-64C37519: G***, kibuzzard-64C37519, B.Cu at (129.2, 108.8)
- added kibuzzard-64C3756D: G***, kibuzzard-64C3756D, B.Cu at (150.1, 109.0)
- added kibuzzard-64C375B4: G***, kibuzzard-64C375B4, B.Cu at (148.1, 117.3)
- added kibuzzard-64C375BE: G***, kibuzzard-64C375BE, B.Cu at (148.1, 115.3)
- added kibuzzard-64C375C5: G***, kibuzzard-64C375C5, B.Cu at (148.1, 113.3)
- added kibuzzard-64C375DA: G***, kibuzzard-64C375DA, B.Cu at (148.1, 111.3)
- added kibuzzard-64C375F2: G***, kibuzzard-64C375F2, B.Cu at (131.3, 111.3)
- added kibuzzard-64C37614: G***, kibuzzard-64C37614, B.Cu at (131.3, 115.3)
- added kibuzzard-64C3761E: G***, kibuzzard-64C3761E, B.Cu at (131.3, 117.3)
- added kibuzzard-64C37A88: G***, kibuzzard-64C37A88, F.Cu at (135.9, 122.9)
- added kibuzzard-64C37A88: G***, kibuzzard-64C37A88, B.Cu at (142.5, 119.4)
- added kibuzzard-64C37A88: G***, kibuzzard-64C37A88, B.Cu at (135.9, 122.9)
- added kibuzzard-64C37AD1: G***, kibuzzard-64C37AD1, F.Cu at (138.4, 122.7)
- added kibuzzard-64C37B05: G***, kibuzzard-64C37B05, B.Cu at (141.0, 122.8)
- added kibuzzard-64C37B2E: G***, kibuzzard-64C37B2E, B.Cu at (138.4, 122.7)
- added kibuzzard-64C37B4E: G***, kibuzzard-64C37B4E, F.Cu at (141.0, 122.8)
- added kibuzzard-64C37B97: G***, kibuzzard-64C37B97, F.Cu at (143.5, 122.9)
- added kibuzzard-64C37BC1: G***, kibuzzard-64C37BC1, B.Cu at (143.5, 122.9)
- added kibuzzard-64C37BF9: G***, kibuzzard-64C37BF9, F.Cu at (146.1, 122.8)
- added kibuzzard-64C37C16: G***, kibuzzard-64C37C16, B.Cu at (146.1, 122.8)
- added kibuzzard-64C37C5C: G***, kibuzzard-64C37C5C, B.Cu at (147.2, 120.0)
- added kibuzzard-64C37CC9: G***, kibuzzard-64C37CC9, B.Cu at (136.3, 119.4)
- added kibuzzard-64C37D63: G***, kibuzzard-64C37D63, B.Cu at (139.7, 116.8)
- added kibuzzard-64C37D9D: G***, kibuzzard-64C37D9D, B.Cu at (139.7, 115.3)
- added kibuzzard-64C37FAB: G***, kibuzzard-64C37FAB, B.Cu at (131.3, 113.3)
- added kibuzzard-64C38090: G***, kibuzzard-64C38090, B.Cu at (129.8, 121.4)
- added kibuzzard-64C3B30F: G***, kibuzzard-64C3B30F, F.Cu at (149.9, 120.7)
- moved JP2 30.3 mm to (150.2, 120.0), turned to 0 degrees
- moved JP8 29.8 mm to (150.2, 117.3)
- moved JP11 27.8 mm to (150.2, 111.3)
- moved JP10 26.5 mm to (150.2, 113.3)
- moved JP9 26.1 mm to (150.2, 115.3)
- moved JP1 21.1 mm to (139.7, 119.4)
- moved JP4 15.1 mm to (129.2, 111.3), turned to 0 degrees
- moved R2 11.4 mm to (131.4, 119.4), turned to 90 degrees
- moved JP3 10.5 mm to (129.8, 119.6), turned to 180 degrees
- moved R3 5.39 mm to (133.3, 119.4), turned to 90 degrees
- moved JP7 2.68 mm to (129.2, 117.3), turned to 0 degrees
- moved R1 1.42 mm to (146.1, 119.4)
- moved C2 0.90 mm to (144.1, 119.4)
- moved C4 0.90 mm to (135.3, 119.4)
- moved C1 0.64 mm to (142.2, 119.4)
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Routing:
- net +3.3V: track 0.00 -> 54.9 mm, vias 0 -> 3
- net SCL: track 0.00 -> 46.7 mm, vias 0 -> 4
- net SDA: track 0.00 -> 45.5 mm, vias 0 -> 3
- net A1: track 0.00 -> 26.5 mm, vias 0 -> 3
- net VDDA: track 0.00 -> 22.9 mm, vias 0 -> 3
- net ~{RESET}: track 0.00 -> 21.1 mm, vias 0 -> 1
- net ~{DRDY}: track 0.00 -> 19.1 mm, vias 0 -> 1
- net A0: track 0.00 -> 17.2 mm, vias 0 -> 1
- net AIN3: track 0.00 -> 17.0 mm
- net AIN0: track 0.00 -> 16.9 mm
- net REFP: track 0.00 -> 16.8 mm, vias 0 -> 1
- net REFN: track 0.00 -> 16.2 mm
- net AIN2: track 0.00 -> 16.0 mm
- net AIN1: track 0.00 -> 16.0 mm
- net GND: track 0.00 -> 10.8 mm, vias 0 -> 20
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- added copper zone on B.Cu, net GND
- added copper zone on F.Cu, net GND
