File: Hardware/Qwiic_ADS1219.kicad_sch (KiCad schematic)
At the start: 30 parts, among them J1 Qwiic_RA, J2 Qwiic_RA, J3 Conn_01x06, J4 Conn_01x06, J5 Conn_01x02, J6 I2C_01x04, U1 ADS1219IPW

Commit message: Routed
Parts:
- added R4, R5: 10k, SparkFun-Resistor:R_0603_1608Metric, symbol SparkFun-Resistor:10k_0603
Connections:
- net +3.3V: now also R4.1, R5.1
- net ~{DRDY}: now also R4.2
- net ~{RESET}: now also R5.2
Other:
- note added: "Open jumper to disable LED"
- moved on the sheet: C1, C2, C3, C4, JP1, JP3, R2, R3, U1
