File: Hardware/SparkX_ADC_ADS1219.kicad_pcb (KiCad board)
At the start: 2 copper layers, 25.4 x 25.4 mm, 75 parts, among them J1 Qwiic_RA, J2 Qwiic_RA, J3 Conn_01x06, J4 Conn_01x06, J5 Conn_01x02, J6 I2C_01x04, U1 ADS1219IPW

Commit message: Rename everything
Parts:
- removed kibuzzard-64C37D9D: G***, kibuzzard-64C37D9D
- added G***: LOGO, SparkFun-Aesthetic:SparkX_Logo_10mm, B.Cu at (139.7, 113.0)
- added kibuzzard-64C3BD7A: G***, kibuzzard-64C3BD7A, B.Cu at (139.7, 115.4)
Routing:
- net SDA: track 45.5 -> 46.6 mm
- net SCL: track 46.7 -> 47.7 mm
- net GND: vias 20 -> 24

Commit message: Add panel
Parts:
- added FID1: Fiducial_0.635, SparkFun-Aesthetic:Fiducial_0.635mm, F.Cu at (151.8, 121.9)
- added FID2: Fiducial_0.635, SparkFun-Aesthetic:Fiducial_0.635mm, B.Cu at (151.8, 121.9)
- added FID3: Fiducial_0.635, SparkFun-Aesthetic:Fiducial_0.635mm, F.Cu at (127.6, 106.7)
- added FID4: Fiducial_0.635, SparkFun-Aesthetic:Fiducial_0.635mm, B.Cu at (127.6, 106.7)
- added U2: ~, SparkFun-Aesthetic:ORDERING_INSTRUCTIONS, F.Cu at (156.9, 76.3)
Connections:
- J1 pad NC1: (no net) -> unconnected-(J1-NC-PadNC1)
- J1 pad NC2: (no net) -> unconnected-(J1-NC-PadNC2)
- J2 pad NC1: (no net) -> unconnected-(J2-NC-PadNC1)
- J2 pad NC2: (no net) -> unconnected-(J2-NC-PadNC2)
Other:
- board text added: "Solder Mask: Black Silkscreen: White Layers: 2 Finish: HASL Lead-free Thickness: 1.6mm Copper weight: 1oz"
