File: Hardware/SparkX_ADC_ADS1219.kicad_sch (KiCad schematic)
At the start: 32 parts, among them J1 Qwiic_RA, J2 Qwiic_RA, J3 Conn_01x06, J4 Conn_01x06, J5 Conn_01x02, J6 I2C_01x04, U1 ADS1219IPW

Commit message: Add panel
Parts:
- added FID1, FID2, FID3, FID4: Fiducial_0.635, SparkFun-Aesthetic:Fiducial_0.635mm, symbol SparkFun-Aesthetic:Fiducial_0.635
- added U2: ~, SparkFun-Aesthetic:ORDERING_INSTRUCTIONS, symbol SparkFun-Aesthetic:Ordering_Instructions
- C1, C3: PROD_ID 7888 -> CAP-07888
- C2, C4: PROD_ID 810 -> CAP-00810
- D1: PROD_ID 819 -> DIO-00819
- J1, J2: PROD_ID 13694 -> CONN-13694
- R1: PROD_ID 7856 -> RES-07856
- R2, R3: PROD_ID 8272 -> RES-08272
- R4, R5: PROD_ID 824 -> RES-00824
- U1: PROD_ID (none) -> IC-19659
Connections:
- new net: J2.NC1 (NC), J2.NC2 (NC)
- new net: J1.NC1 (NC), J1.NC2 (NC)
Other:
- title: Qwiic ADS1219 -> SparkX ADC ADS1219 (Qwiic)
- moved on the sheet: D1, J5, J6, JP2, JP3, R1, R2, R3
